File: midinomad.sch (KiCad schematic (older format))
At the start: 65 parts, among them J1 MIDI IN, J2 MIDI OUT, J3 Nomad 5pin, J4 Nomad 100, J7 DC IN, U1 6N138, U2 L7805, U4 74HC4053

Commit message: Rev. 6 PCB & schematics
Parts:
- removed C4: 0.1uF, Capacitor_THT:C_Disc_D6.0mm_W2.5mm_P5.00mm, symbol pspice:C
- removed R?: 220R, Resistor_THT:R_Axial_DIN0207_L6.3mm_D2.5mm_P10.16mm_Horizontal, symbol Device:R
- removed U4: 74HC4053, Package_DIP:DIP-16_W7.62mm_LongPads, symbol 74xx:74HC4053
- removed U? (x3): MOC3041M, symbol Relay_SolidState:MOC3041M
- added D2, D3, D4: 1N4007, Diode_THT:D_DO-41_SOD81_P10.16mm_Horizontal, symbol Diode:1N4007
- added K1, K2, K3: SANYOU_SRD_Form_C, Relay_THT:Relay_SPDT_SANYOU_SRD_Series_Form_C, symbol Relay:SANYOU_SRD_Form_C
- added Q1, Q2, Q3: 2N2222, Package_TO_SOT_THT:TO-18-3, symbol Transistor_BJT:2N2646
- added R2, R6, R8: 1k, Resistor_THT:R_Axial_DIN0207_L6.3mm_D2.5mm_P10.16mm_Horizontal, symbol Device:R
- U2, U3: renamed from U?; footprint (none) -> Package_DIP:DIP-6_W7.62mm_LongPads
- gave numbers to parts that had none: 2
- renumbered C5 to C3, D4 to D10, D2 to D5, D5 to D6, D3 to D7, D6 to D8, D7 to D9, J3 to J2, J4 to J3, J2 to J4, J7 to J5, R17 to R10, R18 to R11, R19 to R13, R22 to R14, R4 to R15, R7 to R16, R20 to R17, R23 to R18, R13 to R19, R10 to R20, R5 to R21, R8 to R22, R21 to R23, R14 to R25, R11 to R26, R6 to R27, R9 to R28, R15 to R29, R2 to R3, R12 to R30, R3 to R4, R25 to R5, R16 to R7, JP1 to RXJ1, JP2 to TXJ1, U2 to U4
Connections:
- net +2V: now also K1.4, K2.3, K3.4
- net +5V: now also D2.1 (K), D3.1 (K), D4.1 (K), K1.5, K2.5, K3.5
- net -3V: now also K1.3, K2.4, K3.3
- net Arduino_D4: now also R2.2
- net Arduino_D5: now also R8.2
- net Arduino_D6: now also R6.2
- net GNDREF: now also Q1.3 (B1), Q2.3 (B1), Q3.3 (B1)
- net MESA_SWA_(SOLO): now also K1.1
- net MESA_SWB_(REV): now also K2.1
- net MESA_SWC_(EQ): now also K3.1
- new net: D2.2 (A), K1.2, Q1.1 (B2)
- new net: D3.2 (A), K2.2, Q3.1 (B2)
- new net: D4.2 (A), K3.2, Q2.1 (B2)
- new net: Q1.2 (E), R2.1
- new net: Q2.2 (E), R6.1
- new net: Q3.2 (E), R8.1

Commit message: before adding the rest of relays
Parts:
- Q1, Q2, Q3: footprint Package_TO_SOT_THT:TO-18-3 -> Package_TO_SOT_THT:TO-92
Changed lines of the file:
@@
 F 0 "Q1" H 5490 1246 50  0000 L CNN
 F 1 "2N2222" H 5490 1155 50  0000 L CNN
-F 2 "Package_TO_SOT_THT:TO-18-3" H 5500 1125 50  0001 L CIN
+F 2 "Package_TO_SOT_THT:TO-92" H 5500 1125 50  0001 L CIN
 F 3 "http://www.bucek.name/pdf/2n2646,2647.pdf" H 5300 1200 50  0001 L CNN
 	1    5300 1200
@@
 F 0 "Q2" H 7540 2596 50  0000 L CNN
 F 1 "2N2222" H 7540 2505 50  0000 L CNN
-F 2 "Package_TO_SOT_THT:TO-18-3" H 7550 2475 50  0001 L CIN
+F 2 "Package_TO_SOT_THT:TO-92" H 7550 2475 50  0001 L CIN
 F 3 "http://www.bucek.name/pdf/2n2646,2647.pdf" H 7350 2550 50  0001 L CNN
 	1    7350 2550
@@
 F 0 "Q3" H 5540 3046 50  0000 L CNN
 F 1 "2N2222" H 5540 2955 50  0000 L CNN
-F 2 "Package_TO_SOT_THT:TO-18-3" H 5550 2925 50  0001 L CIN
+F 2 "Package_TO_SOT_THT:TO-92" H 5550 2925 50  0001 L CIN
 F 3 "http://www.bucek.name/pdf/2n2646,2647.pdf" H 5350 3000 50  0001 L CNN
 	1    5350 3000
